File: PCB/Audio_Interface.sch (KiCad schematic (older format))
At the start: 6 parts

Commit message: Audio Switch eindesignt
Parts:
- removed K? (x2): G6K-2F-Y-TR_DC5, Artikel:Relais_Omron_G6K-2F-Y, symbol Artikel:G6K-2F-Y-TR_DC5
- added C? (x2): 100n_0603, Kondensator:CAPC1608, symbol Kondensator:100n_0603
- added IC? (x2): TS5A22364, Artikel:SOIC-10, symbol Artikel:TS5A22364
- added R? (x2): 10K_0603, Widerstand:RESC1608, symbol Widerstand:10K_0603
- J1, J2, J3, J4: renamed from J?; NB ?NB? -> (none)
Connections:
- net IN_Left_1: now also IC?.8 (NC2)
- net IN_Left_2: now also IC?.10 (NO2)
- net IN_Right_1: now also IC?.4 (NC1)
- net IN_Right_2: now also IC?.2 (NO1)
- net Input_Select: now also IC?.5 (IN1), IC?.7 (IN2), R?.1
- net OUT_Left_1: now also IC?.8 (NC2)
- net OUT_Left_2: now also IC?.10 (NO2)
- net OUT_Right_1: now also IC?.4 (NC1)
- net OUT_Right_2: now also IC?.2 (NO1)
- net Output_Select: now also IC?.5 (IN1), IC?.7 (IN2), R?.1
- new net +3V3: C?.1, C?.1, IC?.1 (VCC), IC?.1 (VCC)
- new net GND: C?.2, C?.2, IC?.6 (GND), IC?.6 (GND), R?.2, R?.2
- new net Left: IC?.9 (COM2), IC?.9 (COM2)
- new net Right: IC?.3 (COM1), IC?.3 (COM1)
Other:
- note added: "Audio GND darf nicht mit normalen GND verbunden werden!\n"
- note added: "Aux Output 1"
- note added: "Aux Output 2\n"
- note added: "Layout Hinweis\n"
- note added: "Output Selection"
- moved on the sheet: J1, J2, J3, J4

Commit message: Sheet USB
USB Switch und USB Input Stecker hinzugefügt
Parts:
- J1, J2, J3, J4: symbol Stecker:AUX_TRRS -> Stecker:AUX_TRS_SMD
- gave numbers to parts that had none: 6
Connections:
- net GNDA: now also J1.2 (GND), J2.2 (GND), J3.2 (GND), J4.2 (GND); no longer J1.3 (GND), J2.3 (GND), J3.3 (GND), J4.3 (GND)
- net IN_Left_1: now also J1.3 (Left), J1.4 (Left); no longer J1.1 (Left), J1.8 (Left)
- net IN_Left_2: now also J2.3 (Left), J2.4 (Left); no longer J2.1 (Left), J2.8 (Left)
- net IN_Right_1: now also J1.5 (Right); no longer J1.4 (Right), J1.7 (Right)
- net IN_Right_2: now also J2.5 (Right); no longer J2.4 (Right), J2.7 (Right)
- net OUT_Left_1: now also J3.3 (Left), J3.4 (Left); no longer J3.1 (Left), J3.8 (Left)
- net OUT_Left_2: now also J4.3 (Left), J4.4 (Left); no longer J4.1 (Left), J4.8 (Left)
- net OUT_Right_1: now also J3.5 (Right); no longer J3.4 (Right), J3.7 (Right)
- net OUT_Right_2: now also J4.5 (Right); no longer J4.4 (Right), J4.7 (Right)
